File: CLOCK/CLOCK.kicad_sch (KiCad schematic)
At the start: 4 parts

Commit message: WEEK2
WEEK2
Parts:
- removed H1, H2, H3, H4: MountingHole, footprints:MountingHole_3.2mm_M3, symbol HPS:MountingHole
- added C1, C3, C7, C?: C_0805_0.1uf, footprints:C_0805_2012Metric, symbol HPS:C_0805_0.1uf
- added C4, C5: C_0805_22pf, footprints:C_0805_2012Metric, symbol HPS:C_0805_22pf
- added C6: C_0805_1uf, footprints:C_0805_2012Metric, symbol HPS:C_0805_1uf
- added D1: LED_0805, footprints:LED_0805_2012Metric, symbol HPS:LED_0805
- added J1: Conn_01x06, footprints:PinHeader_1x06_P2.54mm_Vertical, symbol HPS:Conn_01x06
- added J2: PJ-102AH, footprints:PJ-102AH, symbol HPS:PJ-102AH
- added R1: R_0805_2.2K, footprints:R_0805_2012Metric, symbol HPS:R_0805_2.2K
- added R2: R_0805_10K, footprints:R_0805_2012Metric, symbol HPS:R_0805_10K
- added R3, R4: R_0805_47, footprints:R_0805_2012Metric, symbol HPS:R_0805_47
- added SW1: Omron_B3F_SPST, footprints:SW_SPST_Omron_B3FS-100xP, symbol HPS:Omron_B3F_SPST
- added U1: ATmega328-PU, footprints:DIP-28_W7.62mm, symbol HPS:ATmega328-PU
- added U2: L7805, symbol HPS:L7805
- added Y1: Crystal_16MHz, footprints:Crystal_SMD_HC49-SD, symbol HPS:Crystal_16MHz
Connections:
- new net: C5.2, U1.10 (XTAL2/PB7), Y1.1
- new net: C4.2, U1.9 (XTAL1/PB6), Y1.2
- new net: D1.1 (K), R1.1
- new net: J1.4 (Pin_4), R4.2
- new net: J1.5 (Pin_5), R3.2
- new net: C3.2, J1.6 (Pin_6)
- new net: C6.1, J2.1 (POLE), U2.1 (IN)
- new net: C1.1, U1.21 (AREF)
- new net GND: C1.2, C4.1, C5.1, C6.2, C7.2, C?.2, J2.2 (OUT), R1.2, SW1.1 (A), SW1.2 (A), U1.22 (GND), U1.8 (GND), U2.2 (GND)
- new net LED_SCK: D1.2 (A), U1.19 (PB5)
- new net RESET: C3.1, R2.2, SW1.3 (B), SW1.4 (B), U1.1 (~{RESET}/PC6)
- new net RXD: R3.1, U1.2 (PD0)
- new net TXD: R4.1, U1.3 (PD1)
- new net VCC: C7.1, C?.1, R2.1, U1.20 (AVCC), U1.7 (VCC), U2.3 (OUT)
Other:
- note added: "LED"
- note added: "MCU"
- note added: "POWER INPUT"
- note added: "SERIAL"
- note added: "Vf = 2v Vr = 3v 10mcd @1.35mA therefore R = 2.2Kohm"
