File: CLOCK/CLOCK.kicad_sch (KiCad schematic)
At the start: 18 parts, among them J1 Conn_01x06, J2 PJ-102AH, SW1 Omron_B3F_SPST, U1 ATmega328-PU, U2 L7805, Y1 Crystal_16MHz

Commit message: WEEK 3
Parts:
- added D1, D2, D3, D4: KWM-30881CVB, footprints:KWM-30881CVB, symbol HPS:KWM-30881CVB
- added U1, U2, U3, U4: MAX7219, footprints:DIP-24_W7.62mm, symbol HPS:MAX7219

Commit message: WEEK4/5
PROGRSSING
Parts:
- removed D2: KWM-30881CVB, footprints:KWM-30881CVB, symbol HPS:KWM-30881CVB
- removed U2, U3, U4: MAX7219, footprints:DIP-24_W7.62mm, symbol HPS:MAX7219
- added BT1: Battery_Cell, footprints:BatteryHolder_Keystone_106_1x20mm, symbol HPS:Battery_Cell
- added C10, C11, C8, C9: C_0805_10uf, footprints:C_0805_2012Metric, symbol HPS:C_0805_10uf
- added C12, C13, C14, C15: C_0805_0.1uf, footprints:C_0805_2012Metric, symbol HPS:C_0805_0.1uf
- added D5: KWM-30881CVB, footprints:KWM-30881CVB, symbol HPS:KWM-30881CVB
- added H1, H2, H3, H4: MountingHole, footprints:MountingHole_3.2mm_M3, symbol HPS:MountingHole
- added J3: Conn_02x03_Odd_Even, footprints:PinHeader_2x03_P2.54mm_Vertical, symbol HPS:Conn_02x03_Odd_Even
- added R10, R9: R_0805_4.7K, footprints:R_0805_2012Metric, symbol HPS:R_0805_4.7K
- added R11, R12, R13, R14, R5, R6, R7: R_0805_10K, footprints:R_0805_2012Metric, symbol HPS:R_0805_10K
- added SW2, SW3, SW4: Omron_B3F_SPST, footprints:SW_SPST_Omron_B3FS-100xP, symbol HPS:Omron_B3F_SPST
- added U3: DS1307_DIP-8, footprints:DIP-8_W7.62mm, symbol HPS:DS1307_DIP-8
- added U5, U6, U7: MAX7219, footprints:DIP-24_W7.62mm, symbol HPS:MAX7219
- added U8: ADT7410, footprints:SOIC-8_3.9x4.9mm_P1.27mm, symbol HPS:ADT7410
- added Y2: Crystal_32768Hz, footprints:Crystal_SMD_2Pin_3.2x1.5mm, symbol HPS:Crystal_32768Hz
- gave numbers to parts that had none: 1
- renumbered D1 to D2, U1 to U4
Connections:
- net GND: now also C5.2, U4.4 (GND), U4.9 (GND), BT1.2 (-), C10.1, C11.1, C12.2, C13.2, C14.2, C15.2, C8.1, C9.1, J3.6 (Pin_6), SW2.1 (A), SW2.2 (A), SW3.1 (A), SW3.2 (A), SW4.1 (A), SW4.2 (A), U3.4 (GND), U5.4 (GND), U5.9 (GND), U6.4 (GND), U6.9 (GND), U7.4 (GND), U7.9 (GND); no longer C5.1
- net LED_SCK: now also J3.3 (Pin_3)
- net RESET: now also R2.1, J3.5 (Pin_5); no longer R2.2
- net VCC: now also R2.2, U4.19 (V+), C10.2, C11.2, C12.1, C13.1, C14.1, C15.1, C8.2, C9.2, J3.2 (Pin_2), R10.1, R11.1, R12.1, R13.1, R14.1, R5.1, R6.1, R7.1, R9.1, U3.8 (VCC), U5.19 (V+), U6.19 (V+), U7.19 (V+); no longer R2.1
- net 1DIG_4: now reaches D2.1 (R5)
- net 1DIG_4: now also U4.3 (DIG_4)
- net 1SEG_C: now reaches D2.10 (C4)
- net 1SEG_C: now also U4.20 (SEG_C)
- net 1SEG_E: now reaches D2.11 (C6)
- net 1SEG_E: now also D2.16 (C8), U4.21 (SEG_E)
- net 1DIG_3: now reaches D2.12 (R4)
- net 1DIG_3: now also U4.7 (DIG_3)
- net 1SEG_DP: now reaches D2.13 (C1)
- net 1SEG_DP: now also U4.22 (SEG_DP)
- net 1DIG_1: now reaches D2.14 (R2)
- net 1DIG_1: now also U4.11 (DIG_1)
- net 1SEG_F: now reaches D2.15 (C7)
- net 1SEG_F: now also U4.15 (SEG_F)
- net 1DIG_6: now reaches D2.2 (R7)
- net 1DIG_6: now also U4.5 (DIG_6)
- net 1SEG_A: now reaches D2.3 (C2)
- net 1SEG_A: now also U4.14 (SEG_A)
- net 1SEG_B: now reaches D2.4 (C3)
- net 1SEG_B: now also U4.16 (SEG_B)
- net 1DIG_7: now reaches D2.5 (R8)
- net 1DIG_7: now also U4.8 (DIG_7)
- net 1SEG_D: now reaches D2.6 (C5)
- net 1SEG_D: now also U4.23 (SEG_D)
- net 1DIG_5: now reaches D2.7 (R6)
- net 1DIG_5: now also U4.10 (DIG_5)
- net 1DIG_2: now reaches D2.8 (R3)
- net 1DIG_2: now also U4.6 (DIG_2)
- net 1DIG_0: now reaches D2.9 (R1)
- net 1DIG_0: now also U4.2 (DIG_0)
- net at U1.10 (XTAL2/PB7), Y1.1: now also C5.1; no longer C5.2
- net 2DIG_4: now reaches D3.1 (R5)
- net 2DIG_4: now also U5.3 (DIG_4)
- net 2SEG_C: now reaches D3.10 (C4)
- net 2SEG_C: now also U5.20 (SEG_C)
- net 2SEG_E: now reaches D3.11 (C6)
- net 2SEG_E: now also D3.16 (C8), U5.21 (SEG_E)
- net 2DIG_3: now reaches D3.12 (R4)
- net 2DIG_3: now also U5.7 (DIG_3)
- net 2SEG_DP: now reaches D3.13 (C1)
- net 2SEG_DP: now also U5.22 (SEG_DP)
- net 2DIG_1: now reaches D3.14 (R2)
- net 2DIG_1: now also U5.11 (DIG_1)
- net 2SEG_F: now reaches D3.15 (C7)
- net 2SEG_F: now also U5.15 (SEG_F)
- net 2DIG_6: now reaches D3.2 (R7)
- net 2DIG_6: now also U5.5 (DIG_6)
- net 2SEG_A: now reaches D3.3 (C2)
- net 2SEG_A: now also U5.14 (SEG_A)
- net 2SEG_B: now reaches D3.4 (C3)
- net 2SEG_B: now also U5.16 (SEG_B)
- net 2DIG_7: now reaches D3.5 (R8)
- net 2DIG_7: now also U5.8 (DIG_7)
- net 2SEG_D: now reaches D3.6 (C5)
- net 2SEG_D: now also U5.23 (SEG_D)
- net 2DIG_5: now reaches D3.7 (R6)
- net 2DIG_5: now also U5.10 (DIG_5)
- net 2DIG_2: now reaches D3.8 (R3)
- net 2DIG_2: now also U5.6 (DIG_2)
- net 2DIG_0: now reaches D3.9 (R1)
- net 2DIG_0: now also U5.2 (DIG_0)
- net CLK: now reaches U1.14 (PB0)
- net CLK: now also U4.13 (CLK), U5.13 (CLK), U6.13 (CLK), U7.13 (CLK)
- net DIN: now reaches U1.15 (PB1)
- net DIN: now also U7.1 (DIN)
- net CS: now reaches U1.16 (PB2)
- net CS: now also U4.12 (LOAD), U5.12 (LOAD), U6.12 (LOAD), U7.12 (LOAD)
- net MOSI: now reaches U1.17 (PB3)
- net MOSI: now also J3.4 (Pin_4)
- net MISO: now reaches U1.18 (PB4)
- net MISO: now also J3.1 (Pin_1)
- net SDA: now reaches U1.27 (PC4)
- net SDA: now also R10.2, U3.5 (SDA)
- net SCL: now reaches U1.28 (PC5)
- net SCL: now also R9.2, U3.6 (SCL)
- net BTN_DWN: now reaches U1.4 (PD2)
- net BTN_DWN: now also R6.2, SW3.3 (B), SW3.4 (B)
- net BTN_SEL: now reaches U1.5 (PD3)
- net BTN_SEL: now also R7.2, SW4.3 (B), SW4.4 (B)
- net BTN_UP: now reaches U1.6 (PD4)
- net BTN_UP: now also R5.2, SW2.3 (B), SW2.4 (B)
- net 3DIG_4: now reaches D4.1 (R5)
- net 3DIG_4: now also U6.3 (DIG_4)
- net 3SEG_C: now reaches D4.10 (C4)
- net 3SEG_C: now also U6.20 (SEG_C)
- net 3SEG_E: now reaches D4.11 (C6)
- net 3SEG_E: now also D4.16 (C8), U6.21 (SEG_E)
- net 3DIG_3: now reaches D4.12 (R4)
- net 3DIG_3: now also U6.7 (DIG_3)
- net 3SEG_DP: now reaches D4.13 (C1)
- net 3SEG_DP: now also U6.22 (SEG_DP)
- net 3DIG_1: now reaches D4.14 (R2)
- net 3DIG_1: now also U6.11 (DIG_1)
- net 3SEG_F: now reaches D4.15 (C7)
- net 3SEG_F: now also U6.15 (SEG_F)
- net 3DIG_6: now reaches D4.2 (R7)
- net 3DIG_6: now also U6.5 (DIG_6)
- net 3SEG_A: now reaches D4.3 (C2)
- net 3SEG_A: now also U6.14 (SEG_A)
- net 3SEG_B: now reaches D4.4 (C3)
- net 3SEG_B: now also U6.16 (SEG_B)
- net 3DIG_7: now reaches D4.5 (R8)
- net 3DIG_7: now also U6.8 (DIG_7)
- net 3SEG_D: now reaches D4.6 (C5)
- net 3SEG_D: now also U6.23 (SEG_D)
- net 3DIG_5: now reaches D4.7 (R6)
- net 3DIG_5: now also U6.10 (DIG_5)
- net 3DIG_2: now reaches D4.8 (R3)
- net 3DIG_2: now also U6.6 (DIG_2)
- net 3DIG_0: now reaches D4.9 (R1)
- net 3DIG_0: now also U6.2 (DIG_0)
- net at U4.1 (DIN): now also U5.24 (DOUT)
- net 1SEG_G: now reaches U4.17 (SEG_G)
- net at U4.18 (ISET): now also R11.2
- net D_OUT: now reaches U4.24 (DOUT)
- new net: U3.2 (X2), Y2.1
- new net: U3.1 (X1), Y2.2
- new net: BT1.1 (+), U3.3 (VBAT)
- new net: R13.2, U6.18 (ISET)
- new net: R14.2, U7.18 (ISET)
- new net: U6.1 (DIN), U7.24 (DOUT)
- new net: U5.1 (DIN), U6.24 (DOUT)
- new net: R12.2, U5.18 (ISET)
- new net 2SEG_G: U5.17 (SEG_G)
- new net 3SEG_G: U6.17 (SEG_G)
- new net 4DIG_0: D5.9 (R1), U7.2 (DIG_0)
- new net 4DIG_1: D5.14 (R2), U7.11 (DIG_1)
- new net 4DIG_2: D5.8 (R3), U7.6 (DIG_2)
- new net 4DIG_3: D5.12 (R4), U7.7 (DIG_3)
- new net 4DIG_4: D5.1 (R5), U7.3 (DIG_4)
- new net 4DIG_5: D5.7 (R6), U7.10 (DIG_5)
- new net 4DIG_6: D5.2 (R7), U7.5 (DIG_6)
- new net 4DIG_7: D5.5 (R8), U7.8 (DIG_7)
- new net 4SEG_A: D5.3 (C2), U7.14 (SEG_A)
- new net 4SEG_B: D5.4 (C3), U7.16 (SEG_B)
- new net 4SEG_C: D5.10 (C4), U7.20 (SEG_C)
- new net 4SEG_D: D5.6 (C5), U7.23 (SEG_D)
- new net 4SEG_DP: D5.13 (C1), U7.22 (SEG_DP)
- new net 4SEG_E: D5.11 (C6), D5.16 (C8), U7.21 (SEG_E)
- new net 4SEG_F: D5.15 (C7), U7.15 (SEG_F)
- new net 4SEG_G: U7.17 (SEG_G)
Other:
- note added: "BUTTONS"
- note added: "DISPLAY"
- note added: "ICSP"
- note added: "LEONARDO'S CLOCK"
- note added: "MECHANICAL"
- note added: "REAL TIME CLOCK"
- note added: "RTC_XTAL1"
- note added: "RTC_XTAL2"
- note added: "SER_RX"
- note added: "SER_TX"
- note added: "VBAT"
- moved on the sheet: C1, C2, C3, C4, C5, C6, C7, D1, D2, J1, J2, R1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
