File: CLOCK/CLOCK.kicad_sch (KiCad schematic)
At the start: 58 parts, among them J1 Conn_01x06, J2 PJ-102AH, J3 Conn_02x03_Odd_Even, SW1 Omron_B3F_SPST, SW2 Omron_B3F_SPST, SW3 Omron_B3F_SPST, SW4 Omron_B3F_SPST, SW5 Omron_B3F_SPST, U1 ATmega328-PU, U2 L7805, U3 DS1307_DIP-8, U4 MAX7219, U5 MAX7219, U6 MAX7219, U7 MAX7219, U8 ADT7410, Y1 Crystal_16MHz, Y2 Crystal_32768Hz

Commit message: WEEK6
UPLOADING PCB
Parts:
- removed J2: PJ-102AH, footprints:PJ-102AH, symbol HPS:PJ-102AH
- added J4: Conn_01x05, footprints:PinHeader_1x05_P2.54mm_Vertical, symbol HPS:Conn_01x05
- added J5: Conn_01x03, footprints:PinHeader_1x03_P2.54mm_Vertical, symbol HPS:Conn_01x03
- added REF**1: Power_inlet_vertical, footprints:Wurth-694106402002, symbol HPS:Power_inlet_vertical
- U2: footprint (none) -> footprints:TO-252-2
- gave numbers to parts that had none: 1
Connections:
- net GND: now also J5.3 (Pin_3), REF**1.2 (OUT)
- net VCC: now also J5.2 (Pin_2)
- net at J1.1 (Pin_1): now also C3.2
- net at J1.4 (Pin_4): no longer R4.2
- net at J1.6 (Pin_6): now also R4.2; no longer C3.2
- net at C6.1, U2.1 (IN): now also REF**1.1 (POLE)
- net PD6: now reaches U1.12 (PD6)
- net PD6: now also J4.1 (Pin_1)
- net PD7: now reaches U1.13 (PD7)
- net PD7: now also J5.1 (Pin_1)
- net PC0: now reaches U1.23 (PC0)
- net PC0: now also J4.2 (Pin_2)
- net PC1: now reaches U1.24 (PC1)
- net PC1: now also J4.3 (Pin_3)
- net PC2: now reaches U1.25 (PC2)
- net PC2: now also J4.4 (Pin_4)
- net PC3: now reaches U1.26 (PC3)
- net PC3: now also J4.5 (Pin_5)
- net D_OUT: no longer names the net of U4.24 (DOUT)
- no-connect marks 6 -> 8
Other:
- note added: "DEBUGGER"
- moved on the sheet: C3, D1, H1, H2, H3, H4, J1, J3, R1, R3, R4, R5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

Commit message: GERBER OUT
LLV-BOARD
Parts:
- added TP1, TP4, TP5, TP6, TP7, TP8, TP9: TestPoint, footprints:TestPoint_THTPad_D2.0mm_Drill1.0mm, symbol HPS:TestPoint
Connections:
- net CLK: now also U1.15 (PB1), TP4.1; no longer U1.14 (PB0)
- net GND: now also TP1.1
- net SCL: now also TP8.1
- net SDA: now also TP7.1
- net VCC: now also R12.2, R13.2, R14.2, TP9.1; no longer R12.1, R13.1, R14.1
- net at U6.18 (ISET): now also R13.1; no longer R13.2
- net at U7.18 (ISET): now also R14.1; no longer R14.2
- net at U5.18 (ISET): now also R12.1; no longer R12.2
- net CS renamed DLOAD
- net DLOAD: now also U1.14 (PB0), TP6.1; no longer U1.16 (PB2)
- net DIN renamed DDATA
- net DDATA: now also U1.16 (PB2), TP5.1; no longer U1.15 (PB1)
Other:
- moved on the sheet: R11, R12, R13, R14

Commit message: GERBER OUT
FINAL COMMIT
Parts:
- U3: renamed from U2; Digikey PN (none) -> 497-7255-1-ND; MFG (none) -> STMicroelectronics; MPN (none) -> L7805CDT-TR
- renumbered C2 to C1, C13 to C10, C9 to C11, C14 to C12, C10 to C13, C15 to C14, C11 to C15, C1 to C2, C12 to C6, C8 to C7, C6 to C8, C7 to C9, D2 to D1, D3 to D2, D4 to D3, D1 to D4, J4 to J2, J5 to J3, REF**1 to J4, J3 to J5, R4 to R1, R14 to R10, R8 to R11, R7 to R12, R6 to R13, R5 to R14, R3 to R2, R9 to R3, R2 to R4, R10 to R5, R11 to R6, R12 to R7, R13 to R8, R1 to R9, SW5 to SW2, SW4 to SW3, SW3 to SW4, SW2 to SW5, TP9 to TP2, TP4 to TP3, TP5 to TP4, TP6 to TP5, TP8 to TP6, U4 to U2, U5 to U4, U6 to U5, U3 to U6
Connections:
- net GND: now also J1.1 (Pin_1), J1.2 (Pin_2)
- net at C3.2: now also J1.6 (Pin_6); no longer J1.1 (Pin_1)
- net at J1.4 (Pin_4): now also R1.2
- no-connect marks 8 -> 6
Other:
- moved on the sheet: C10, C11, C12, C13, C14, C15, C3, C6, C7, R1, R10, R6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
