File: CLOCK/CLOCK.kicad_pcb (KiCad board)
At the start: 2 copper layers, 140 x 90 mm, 58 parts, among them J1 Conn_01x06, J2 PJ-102AH, J3 Conn_02x03_Odd_Even, SW1 Omron_B3F_SPST, SW2 Omron_B3F_SPST, SW3 Omron_B3F_SPST, SW4 Omron_B3F_SPST, U1 ATmega328-PU, U3 DS1307_DIP-8, U4 MAX7219, U5 MAX7219, U6 MAX7219, U7 MAX7219, U8 ADT7410, Y1 Crystal_16MHz, Y2 Crystal_32768Hz

Commit message: FINAL DESIGN
TIME TO ROUTE :)
Parts:
- moved J3 7.62 mm to (127.0, 134.6)
Changed lines of the file:
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@@
   )
   (footprint "footprints:PinHeader_2x03_P2.54mm_Vertical" (layer "F.Cu")
-    (at 119.38 134.62 90)
+    (at 127 134.62 90)
     (descr "Through hole straight pin header, 2x03, 2.54mm pitch, double rows")
     (tags "Through hole pin header THT 2x03 2.54mm double row")

Commit message: WEEK6
UPLOADING PCB
Parts:
- removed the H1 at (85.0, 60.0)
- removed the H2 at (215.0, 60.0)
- removed the H3 at (85.0, 140.0)
- removed the H4 at (215.0, 140.0)
- removed J2: PJ-102AH, footprints:PJ-102AH
- added C16: C_0805_0.1uf, footprints:C_0805_2012Metric, F.Cu at (190.0, 120.0)
- added J4: Conn_01x05, footprints:PinHeader_1x05_P2.54mm_Vertical, F.Cu at (157.5, 139.7)
- added J5: Conn_01x03, footprints:PinHeader_1x03_P2.54mm_Vertical, F.Cu at (153.4, 139.7)
- added R8: R_0805_10K, footprints:R_0805_2012Metric, F.Cu at (159.9, 61.2)
- added REF**1: Power_inlet_vertical, footprints:Wurth-694106402002, B.Cu at (88.9, 128.5)
- added SW5: Omron_B3F_SPST, footprints:SW_SPST_Omron_B3FS-100xP, F.Cu at (166.7, 61.2)
- added U2: L7805, footprints:TO-252-2, F.Cu at (99.1, 136.0)
- moved C6 104.1 mm to (104.1, 139.7), turned to -90 degrees
- moved C7 104.1 mm to (94.0, 139.7), turned to -90 degrees
- moved R5 99.8 mm to (92.3, 61.2), turned to 90 degrees
- moved SW2 99.0 mm to (99.0, 61.2)
- moved BT1 92.5 mm to (205.2, 139.1), turned to 90 degrees
- moved SW4 87.1 mm to (132.7, 61.2)
- moved R7 86.3 mm to (126.0, 61.2), turned to 90 degrees
- moved SW3 77.0 mm to (200.7, 61.2)
- moved U3 75.8 mm to (187.0, 140.0), turned to 180 degrees
- moved Y2 73.7 mm to (192.0, 139.7), turned to -90 degrees
- moved R6 71.1 mm to (193.9, 61.2), turned to 90 degrees
- moved SW1 68.4 mm to (114.3, 137.0), turned to 0 degrees
- moved R9 54.1 mm to (175.3, 134.6), turned to 0 degrees
- moved R10 53.0 mm to (175.3, 137.2), turned to 0 degrees
- moved U8 27.1 mm to (184.0, 121.0)
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Connections:
- D2 pad 16: 1SEG_E -> 1SEG_G
- D3 pad 16: 2SEG_E -> 2SEG_G
- D4 pad 16: 3SEG_E -> 3SEG_G
- D5 pad 16: 4SEG_E -> 4SEG_G
- J1 pad 1: unconnected-(J1-Pad1) -> Net-(C3-Pad2)
- J1 pad 4: Net-(J1-Pad4) -> unconnected-(J1-Pad4)
- J1 pad 6: Net-(C3-Pad2) -> Net-(J1-Pad6)
- R4 pad 2: Net-(J1-Pad4) -> Net-(J1-Pad6)
- U1 pad 11: unconnected-(U1-Pad11) -> BTN_MODE
- U1 pad 12: unconnected-(U1-Pad12) -> PD6
- U1 pad 13: unconnected-(U1-Pad13) -> PD7
- U1 pad 23: unconnected-(U1-Pad23) -> PC0
- U1 pad 24: unconnected-(U1-Pad24) -> PC1
- U1 pad 25: unconnected-(U1-Pad25) -> PC2
- U1 pad 26: unconnected-(U1-Pad26) -> PC3
- U8 pad 1: unconnected-(U8-Pad1) -> SCL
- U8 pad 2: unconnected-(U8-Pad2) -> SDA
- U8 pad 3: unconnected-(U8-Pad3) -> GND
- U8 pad 4: unconnected-(U8-Pad4) -> GND
- U8 pad 7: unconnected-(U8-Pad7) -> GND
- U8 pad 8: unconnected-(U8-Pad8) -> VCC
Routing:
- net CLK: track 0.00 -> 171.5 mm
- net CS: track 0.00 -> 149.7 mm
- net GND: track 0.00 -> 136.0 mm, vias 0 -> 8
- net BTN_UP: track 0.00 -> 116.5 mm, vias 0 -> 2
- net BTN_DWN: track 0.00 -> 94.5 mm, vias 0 -> 1
- net BTN_MODE: track 0.00 -> 93.5 mm, vias 0 -> 2
- net BTN_SEL: track 0.00 -> 90.7 mm, vias 0 -> 1
- net RESET: track 0.00 -> 85.6 mm, vias 0 -> 2
- net DIN: track 0.00 -> 63.0 mm, vias 0 -> 2
- net Net-(U4-Pad1): track 0.00 -> 53.7 mm
- net Net-(U6-Pad1): track 0.00 -> 49.9 mm
- net Net-(U5-Pad1): track 0.00 -> 46.9 mm
- net 1DIG_5: track 0.00 -> 45.2 mm
- net 4DIG_6: track 0.00 -> 45.0 mm
- net 1DIG_6: track 0.00 -> 44.2 mm
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- added copper zone on B.Cu, net GND
- added copper zone on F.Cu, net VCC
Other:
- board text added: "*"
- board text added: "2022"
- board text added: "DECISION"
- board text added: "FE"
- board text added: "GOD BRINGS OPPORTUNITIES, YOU DECIDE WHEN TO TAKE ACTION"
- board text added: "GOOGLE HARDWARE PRODUCT SPRINT"
- board text added: "ILUSION"
- board text added: "LLV"

Commit message: GERBER OUT
LLV-BOARD
Parts:
- added CLK: TestPoint, footprints:TestPoint_THTPad_D2.0mm_Drill1.0mm, F.Cu at (143.3, 111.8)
- added DDATA: TestPoint, footprints:TestPoint_THTPad_D2.0mm_Drill1.0mm, F.Cu at (179.8, 114.8)
- added DLOAD: TestPoint, footprints:TestPoint_THTPad_D2.0mm_Drill1.0mm, F.Cu at (214.4, 111.3)
- added G***: LOGO, footprints:HPS_logo, B.Cu at (117.3, 116.3)
- added GND: TestPoint, footprints:TestPoint_THTPad_D2.0mm_Drill1.0mm, F.Cu at (126.2, 138.9)
- added SCL: TestPoint, footprints:TestPoint_THTPad_D2.0mm_Drill1.0mm, F.Cu at (185.9, 114.8)
- added SDA: TestPoint, footprints:TestPoint_THTPad_D2.0mm_Drill1.0mm, F.Cu at (189.5, 115.3)
- added VCC: TestPoint, footprints:TestPoint_THTPad_D2.0mm_Drill1.0mm, F.Cu at (120.1, 138.9)
- moved R7 71.2 mm to (197.1, 58.2), turned to 180 degrees
- moved SELECT 64.4 mm to (197.1, 63.0)
- moved MODE 63.9 mm to (102.9, 63.0)
- moved R8 57.1 mm to (102.9, 58.4), turned to 180 degrees
- moved R5 42.2 mm to (134.4, 58.4), turned to 180 degrees
- moved UP 35.4 mm to (134.4, 63.0)
- moved DOWN 35.1 mm to (165.6, 63.0)
- moved R6 28.5 mm to (165.6, 58.2), turned to 180 degrees
- moved REF**1 24.4 mm to (113.3, 127.5), turned to 90 degrees
- moved RESET 13.6 mm to (124.5, 128.0)
- moved Y2 6.61 mm to (192.3, 133.1)
- moved U3 6.06 mm to (189.2, 134.4)
- moved D2 4.01 mm to (102.9, 83.1)
- moved R1 3.99 mm to (141.5, 136.3), turned to 90 degrees
- moved D5 3.71 mm to (197.1, 83.1)
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- renumbered SW3 to DOWN, SW5 to MODE, SW1 to RESET, SW4 to SELECT, SW2 to UP
Connections:
- R12 pad 1: VCC -> Net-(U5-Pad18)
- R12 pad 2: Net-(R12-Pad2) -> VCC
- R13 pad 1: VCC -> Net-(U6-Pad18)
- R13 pad 2: Net-(R13-Pad2) -> VCC
- R14 pad 1: VCC -> Net-(U7-Pad18)
- R14 pad 2: Net-(R14-Pad2) -> VCC
- U1 pad 14: CLK -> DLOAD
- U1 pad 15: DIN -> CLK
- U1 pad 16: CS -> DDATA
- U4 pad 12: CS -> DLOAD
- U4 pad 24: D_OUT -> unconnected-(U4-Pad24)
- U5 pad 12: CS -> DLOAD
- U5 pad 18: Net-(R12-Pad2) -> Net-(U5-Pad18)
- U6 pad 12: CS -> DLOAD
- U6 pad 18: Net-(R13-Pad2) -> Net-(U6-Pad18)
- U7 pad 1: DIN -> DDATA
- U7 pad 12: CS -> DLOAD
- U7 pad 18: Net-(R14-Pad2) -> Net-(U7-Pad18)
Routing:
- net CS: track 149.7 -> 0.00 mm
- net DLOAD: track 0.00 -> 146.4 mm
- net DDATA: track 0.00 -> 67.3 mm, vias 0 -> 2
- net DIN: track 63.0 -> 0.00 mm, vias 2 -> 0
- net BTN_UP: track 116.5 -> 80.5 mm, vias 2 -> 1
- net Net-(R13-Pad2): track 14.3 -> 0.00 mm
- net Net-(R12-Pad2): track 11.7 -> 0.00 mm
- net Net-(U7-Pad18): track 0.00 -> 11.6 mm
- net Net-(R14-Pad2): track 11.6 -> 0.00 mm
- net Net-(U6-Pad18): track 0.00 -> 11.5 mm
- net Net-(U5-Pad18): track 0.00 -> 10.7 mm
- net SDA: track 37.2 -> 47.1 mm
- net CLK: track 171.5 -> 180.3 mm
- net BTN_DWN: track 94.5 -> 86.6 mm
- net RESET: track 85.6 -> 78.0 mm
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Other:
- board text added: "21"
- board text added: "AMOR"
- board text added: "FAMILIA"
- board text added: "GILBERTO*LAURA*BERNICE"
- board text added: "GND"
- board text added: "HONOR"
- board text added: "JUNE-AUGUST 2022"
- board text added: "LOVE"
- board text added: "LUJAN VILLASANA"
- board text added: "PANUCO,ZACATECAS"
- board text added: "PC0"
- board text added: "PC1"
- board text added: "PC2"
- board text added: "PC3"
- board text added: "PD6"
- board text added: "PD7"
- board text added: "RESPETO"
- board text added: "RIVERSIDE,CALIFORNIA"
- board text added: "TRUTH,LOYALTY,WISDOM"
- board text added: "VCC"
- board text added: "YOURSELF"
- board text removed: "2022"

Commit message: GERBER OUT
FINAL COMMIT
Parts:
- moved R11 16.9 mm to (119.1, 63.0), turned to 90 degrees
- moved SELECT 10.1 mm to (187.0, 63.0)
- moved MODE 9.13 mm to (112.0, 63.0)
- moved R14 7.42 mm to (128.5, 63.0), turned to 90 degrees
- moved R13 5.85 mm to (168.9, 63.0), turned to 90 degrees
- moved R12 5.71 mm to (194.1, 63.0), turned to 90 degrees
- moved DOWN 3.61 mm to (162.0, 63.0)
- moved C3 3.05 mm to (171.4, 124.0)
- moved UP 2.63 mm to (137.0, 63.0)
- moved R4 1.78 mm to (171.4, 126.2)
- moved D1 1.10 mm to (101.8, 82.8)
- moved D5 1.03 mm to (198.1, 82.8)
- moved D2 0.53 mm to (133.9, 82.8)
- moved D3 0.47 mm to (166.0, 82.8)
- renumbered C2 to C1, C13 to C10, C9 to C11, C14 to C12, C10 to C13, C15 to C14, C11 to C15, C1 to C2, C12 to C6, C8 to C7, C6 to C8, C7 to C9, D2 to D1, D3 to D2, D4 to D3, D1 to D4, DDATA to DATA, J4 to J2, J5 to J3, REF**1 to J4, J3 to J5, DLOAD to LOAD, R4 to R1, R14 to R10, R8 to R11, R7 to R12, R6 to R13, R5 to R14, R3 to R2, R9 to R3, R2 to R4, R10 to R5, R11 to R6, R12 to R7, R13 to R8, R1 to R9, RESET to SW1, U4 to U2, U2 to U3, U5 to U4, U6 to U5, U3 to U6
Connections:
- J1 pad 1: Net-(C3-Pad2) -> GND
- J1 pad 2: unconnected-(J1-Pad2) -> GND
- J1 pad 4: unconnected-(J1-Pad4) -> Net-(J1-Pad4)
- J1 pad 6: Net-(J1-Pad6) -> Net-(C3-Pad2)
- R1 pad 2: Net-(J1-Pad6) -> Net-(J1-Pad4)
Routing:
- net VCC: track 3.36 -> 22.4 mm, vias 0 -> 4
- net Net-(J1-Pad4): track 0.00 -> 8.84 mm
- net 4SEG_DP: track 25.7 -> 34.0 mm
- net 2SEG_DP: track 30.9 -> 38.2 mm
- net Net-(C3-Pad2): track 4.01 -> 11.3 mm
- net 3SEG_DP: track 28.5 -> 35.6 mm
- net 4DIG_7: track 38.6 -> 32.7 mm
- net 3SEG_E: track 22.9 -> 28.7 mm
- net 4SEG_D: track 20.9 -> 15.2 mm
- net 4SEG_E: track 21.6 -> 27.0 mm
- net 4SEG_C: track 17.9 -> 22.9 mm
- net BTN_SEL: track 95.3 -> 90.8 mm
- net 3SEG_C: track 19.8 -> 24.2 mm
- net 4DIG_0: track 28.0 -> 32.4 mm
- net 3DIG_0: track 33.3 -> 37.5 mm
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Other:
- board text added: ":)"
- board text added: "TIME BRINGS FOCUS"
- board text added: "TRUTH*LOYALTY*WISDOM"
- board text removed: "LOVE"
- board text removed: "TRUTH,LOYALTY,WISDOM"
- board text removed: "YOURSELF"
