File: CLOCK/_autosave-CLOCK.kicad_sch (KiCad schematic)
At the start: 58 parts, among them J1 Conn_01x06, J2 PJ-102AH, J3 Conn_02x03_Odd_Even, SW1 Omron_B3F_SPST, SW2 Omron_B3F_SPST, SW3 Omron_B3F_SPST, SW4 Omron_B3F_SPST, SW5 Omron_B3F_SPST, U1 ATmega328-PU, U2 L7805, U3 DS1307_DIP-8, U4 MAX7219, U5 MAX7219, U6 MAX7219, U7 MAX7219, U8 ADT7410, Y1 Crystal_16MHz, Y2 Crystal_32768Hz

Commit message: FINAL DESIGN
TIME TO ROUTE :)
Parts:
- added J4: Conn_01x06, footprints:PinHeader_1x06_P2.54mm_Vertical, symbol HPS:Conn_01x06
Connections:
- net PD6: now reaches U1.12 (PD6)
- net PD6: now also J4.5 (Pin_5)
- net PD7: now reaches U1.13 (PD7)
- net PD7: now also J4.6 (Pin_6)
- net PC0: now reaches U1.23 (PC0)
- net PC0: now also J4.1 (Pin_1)
- net PC1: now reaches U1.24 (PC1)
- net PC1: now also J4.2 (Pin_2)
- net PC2: now reaches U1.25 (PC2)
- net PC2: now also J4.3 (Pin_3)
- net PC3: now reaches U1.26 (PC3)
- net PC3: now also J4.4 (Pin_4)
Other:
- moved on the sheet: D1, H1, H2, H3, H4, J3, R1, R5, R6, R7, R8, SW2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
